Commit message: 更新夹爪链接的碰撞几何体，添加新的盒状碰撞体

File: robot_description/nero_description/urdf/nero_with_gripper.urdf (robot description, URDF)
Before this commit: robot nero_description, 13 links, 12 joints
Links:
- link gripper_left_finger: geometry collision box size=0.0105 0.04 0.004; collision box size=0.036 0.03 0.004
- link gripper_right_finger: geometry collision box size=0.0105 0.04 0.004; collision box size=0.036 0.03 0.004
